File: BPS-CurrentScrutineeringPCB.kicad_pcb (KiCad board)
At the start: 2 copper layers, 38.8 x 33 mm, 9 parts, among them J1 Discharge V_In, J2 Charge V_In, J3 Conn_01x05, J4 Conn_01x05

Commit message: poop
Routing:
- net /V_In+: track 33.9 -> 33.4 mm
Other:
- board text added: "BPS Current Scrutineering PCB"
- board text added: "Charge V_In"
- board text added: "Day Fixed"
- board text added: "Discharge V_In"
